File: 01.pcb/sample.kicad_pcb (KiCad board)
At the start: 2 copper layers, 150.5 x 127.8 mm, 32 parts, among them J4 Conn_01x01, SW2 SW_PUSH

Commit message: 3D
Parts:
- removed J4 (x4): Conn_01x01, SWAN_KEYBOARD:M2hole
Other:
- outline, holes or cut-outs redrawn
- board text added: "1.25"
- board text added: "1.5"
Changed lines of the file:
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@@
   (general
     (thickness 1.6)
-    (drawings 19)
+    (drawings 26)
     (tracks 0)
     (zones 0)
-    (modules 32)
+    (modules 28)
     (nets 1)
   )
@@
     (fp_line (start 7 -7) (end 7 7) (layer Edge.Cuts) (width 0.15))
   )
-  (module SWAN_KEYBOARD:M2hole (layer F.Cu)
-    (at 178.45 31.735)
-    (descr "Mounting Hole 2.2mm, M2")
-    (tags "mounting hole 2.2mm m2")
-    (fp_text reference J4 (at 0 -3.2) (layer F.SilkS) hide
-      (effects (font (size 1 1) (thickness 0.15)))
-    )
-    (fp_text value Conn_01x01 (at 0 3.2) (layer F.Fab)
-      (effects (font (size 1 1) (thickness 0.15)))
-    )
-    (fp_circle (center 0 0) (end 2.45 0) (layer F.CrtYd) (width 0.05))
-    (fp_circle (center 0 0) (end 2.2 0) (layer Cmts.User) (width 0.15))
-    (pad 1 thru_hole circle (at 0 0) (size 3.47 3.47) (drill 2.2) (layers *.Cu *.Mask))
-  )
-  (module SWAN_KEYBOARD:M2hole (layer F.Cu)
-    (at 187.34 143.495)
-    (descr "Mounting Hole 2.2mm, M2")
-    (tags "mounting hole 2.2mm m2")
-    (fp_text reference J4 (at 0 -3.2) (layer F.SilkS) hide
-      (effects (font (size 1 1) (thickness 0.15)))
-    )
-    (fp_text value Conn_01x01 (at 0 3.2) (layer F.Fab)
-      (effects (font (size 1 1) (thickness 0.15)))
-    )
-    (fp_circle (center 0 0) (end 2.45 0) (layer F.CrtYd) (width 0.05))
-    (fp_circle (center 0 0) (end 2.2 0) (layer Cmts.User) (width 0.15))
-    (pad 1 thru_hole circle (at 0 0) (size 3.47 3.47) (drill 2.2) (layers *.Cu *.Mask))
-  )
-  (module SWAN_KEYBOARD:M2hole (layer F.Cu)
-    (at 84.47 123.175)
-    (descr "Mounting Hole 2.2mm, M2")
-    (tags "mounting hole 2.2mm m2")
-    (fp_text reference J4 (at 0 -3.2) (layer F.SilkS) hide
-      (effects (font (size 1 1) (thickness 0.15)))
-    )
-    (fp_text value Conn_01x01 (at 0 3.2) (layer F.Fab)
-      (effects (font (size 1 1) (thickness 0.15)))
-    )
-    (fp_circle (center 0 0) (end 2.45 0) (layer F.CrtYd) (width 0.05))
-    (fp_circle (center 0 0) (end 2.2 0) (layer Cmts.User) (width 0.15))
-    (pad 1 thru_hole circle (at 0 0) (size 3.47 3.47) (drill 2.2) (layers *.Cu *.Mask))
-  )
   (module SWAN_KEYBOARD:Switch_Cuts (layer F.Cu)
     (at 188.61 128.255 330)
@@
     (fp_line (start 7 -7) (end 7 7) (layer Edge.Cuts) (width 0.15))
   )
-  (module SWAN_KEYBOARD:M2hole (layer F.Cu)
-    (at 77.485 38.72)
-    (descr "Mounting Hole 2.2mm, M2")
-    (tags "mounting hole 2.2mm m2")
-    (fp_text reference J4 (at 0 -3.2) (layer F.SilkS) hide
-      (effects (font (size 1 1) (thickness 0.15)))
-    )
-    (fp_text value Conn_01x01 (at 0 3.2) (layer F.Fab)
-      (effects (font (size 1 1) (thickness 0.15)))
-    )
-    (fp_circle (center 0 0) (end 2.2 0) (layer Cmts.User) (width 0.15))
-    (fp_circle (center 0 0) (end 2.45 0) (layer F.CrtYd) (width 0.05))
-    (pad 1 thru_hole circle (at 0 0) (size 3.47 3.47) (drill 2.2) (layers *.Cu *.Mask))
-  )
+  (gr_text 1.5 (at 203.215 140.955) (layer Dwgs.User)
+    (effects (font (size 1.5 1.5) (thickness 0.3)))
+  )
+  (gr_text 1.25 (at 189.88 125.08) (layer Dwgs.User)
+    (effects (font (size 1.5 1.5) (thickness 0.3)))
+  )
+  (gr_text 1.25 (at 146.7 118.73) (layer Dwgs.User)
+    (effects (font (size 1.5 1.5) (thickness 0.3)))
+  )
+  (gr_circle (center 187.34 143.495) (end 188.44 143.495) (layer Edge.Cuts) (width 0.2))
+  (gr_circle (center 84.47 123.175) (end 85.57 123.175) (layer Edge.Cuts) (width 0.2))
+  (gr_circle (center 178.45 31.735) (end 179.55 31.735) (layer Edge.Cuts) (width 0.2))
+  (gr_circle (center 77.485 38.72) (end 78.585 38.72) (layer Edge.Cuts) (width 0.2))
   (gr_arc (start 161.686 177.15) (end 204.612 140.066) (angle -65.01583871) (layer Dwgs.User) (width 0.2))
   (gr_text "Designed by\n   @swan_match" (at 129.682 126.35) (layer B.SilkS)

Commit message: hogy
Parts:
- added J4: Conn_01x01, SWAN_KEYBOARD:M2hole, F.Cu at (178.4, 31.7)
- added J4: Conn_01x01, SWAN_KEYBOARD:M2hole, F.Cu at (187.3, 143.5)
- added J4: Conn_01x01, SWAN_KEYBOARD:M2hole, F.Cu at (84.5, 123.2)
- added J4: Conn_01x01, SWAN_KEYBOARD:M2hole, F.Cu at (77.5, 38.7)
- moved SW2 0.25 mm to (203.8, 140.3)
Routing:
- added copper zone on B.Cu, net GND
- added copper zone on F.Cu, net GND
- removed copper zone on B.Cu, net (none)
- removed copper zone on F.Cu, net (none)
Other:
- outline, holes or cut-outs redrawn
Changed lines of the file:
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@@
   (general
     (thickness 1.6)
-    (drawings 26)
+    (drawings 22)
     (tracks 0)
     (zones 0)
-    (modules 28)
-    (nets 1)
+    (modules 32)
+    (nets 2)
   )
   (page A4)
@@
   )
   (net 0 "")
+  (net 1 GND)
   (net_class Default "これはデフォルトのネット クラスです。"
     (clearance 0.2)
@@
     (uvia_dia 0.3)
     (uvia_drill 0.1)
-  )
-  (module SWAN_KEYBOARD:Switch_Cuts (layer F.Cu)
-    (at 203.85 140.066 330)
+    (add_net GND)
+  )
+  (module SWAN_KEYBOARD:Switch_Cuts (layer F.Cu)
+    (at 203.85 140.32 330)
     (fp_text reference SW2 (at 7.1 8.2 150) (layer F.SilkS) hide
       (effects (font (size 1 1) (thickness 0.15)))
@@
     (fp_line (start -7 -7) (end 7 -7) (layer Edge.Cuts) (width 0.15))
     (fp_line (start 7 -7) (end 7 7) (layer Edge.Cuts) (width 0.15))
+  )
+  (module SWAN_KEYBOARD:M2hole (layer F.Cu)
+    (at 178.45 31.735)
+    (descr "Mounting Hole 2.2mm, M2")
+    (tags "mounting hole 2.2mm m2")
+    (fp_text reference J4 (at 0 -3.2) (layer F.SilkS) hide
+      (effects (font (size 1 1) (thickness 0.15)))
+    )
+    (fp_text value Conn_01x01 (at 0 3.2) (layer F.Fab)
+      (effects (font (size 1 1) (thickness 0.15)))
+    )
+    (fp_circle (center 0 0) (end 2.45 0) (layer F.CrtYd) (width 0.05))
+    (fp_circle (center 0 0) (end 2.2 0) (layer Cmts.User) (width 0.15))
+    (pad 1 thru_hole circle (at 0 0) (size 3.47 3.47) (drill 2.2) (layers *.Cu *.Mask)
+      (net 1 GND))
+  )
+  (module SWAN_KEYBOARD:M2hole (layer F.Cu)
+    (at 187.34 143.495)
+    (descr "Mounting Hole 2.2mm, M2")
+    (tags "mounting hole 2.2mm m2")
+    (fp_text reference J4 (at 0 -3.2) (layer F.SilkS) hide
+      (effects (font (size 1 1) (thickness 0.15)))
+    )
+    (fp_text value Conn_01x01 (at 0 3.2) (layer F.Fab)
+      (effects (font (size 1 1) (thickness 0.15)))
+    )
+    (fp_circle (center 0 0) (end 2.45 0) (layer F.CrtYd) (width 0.05))
+    (fp_circle (center 0 0) (end 2.2 0) (layer Cmts.User) (width 0.15))
+    (pad 1 thru_hole circle (at 0 0) (size 3.47 3.47) (drill 2.2) (layers *.Cu *.Mask)
+      (net 1 GND))
+  )
+  (module SWAN_KEYBOARD:M2hole (layer F.Cu)
+    (at 84.47 123.175)
+    (descr "Mounting Hole 2.2mm, M2")
+    (tags "mounting hole 2.2mm m2")
+    (fp_text reference J4 (at 0 -3.2) (layer F.SilkS) hide
+      (effects (font (size 1 1) (thickness 0.15)))
+    )
+    (fp_text value Conn_01x01 (at 0 3.2) (layer F.Fab)
+      (effects (font (size 1 1) (thickness 0.15)))
+    )
+    (fp_circle (center 0 0) (end 2.45 0) (layer F.CrtYd) (width 0.05))
+    (fp_circle (center 0 0) (end 2.2 0) (layer Cmts.User) (width 0.15))
+    (pad 1 thru_hole circle (at 0 0) (size 3.47 3.47) (drill 2.2) (layers *.Cu *.Mask)
+      (net 1 GND))
   )
   (module SWAN_KEYBOARD:Switch_Cuts (layer F.Cu)
@@
     (fp_line (start 7 -7) (end 7 7) (layer Edge.Cuts) (width 0.15))
   )
-  (gr_text 1.5 (at 203.215 140.955) (layer Dwgs.User)
+  (module SWAN_KEYBOARD:M2hole (layer F.Cu)
+    (at 77.485 38.72)
+    (descr "Mounting Hole 2.2mm, M2")
+    (tags "mounting hole 2.2mm m2")
+    (fp_text reference J4 (at 0 -3.2) (layer F.SilkS) hide
+      (effects (font (size 1 1) (thickness 0.15)))
+    )
+    (fp_text value Conn_01x01 (at 0 3.2) (layer F.Fab)
+      (effects (font (size 1 1) (thickness 0.15)))
+    )
+    (fp_circle (center 0 0) (end 2.2 0) (layer Cmts.User) (width 0.15))
+    (fp_circle (center 0 0) (end 2.45 0) (layer F.CrtYd) (width 0.05))
+    (pad 1 thru_hole circle (at 0 0) (size 3.47 3.47) (drill 2.2) (layers *.Cu *.Mask)
+      (net 1 GND))
+  )
+  (gr_text 1.5 (at 205.755 137.78) (layer F.CrtYd)
     (effects (font (size 1.5 1.5) (thickness 0.3)))
   )
-  (gr_text 1.25 (at 189.88 125.08) (layer Dwgs.User)
+  (gr_text 1.25 (at 189.245 126.35) (layer F.CrtYd)
     (effects (font (size 1.5 1.5) (thickness 0.3)))
   )
-  (gr_text 1.25 (at 146.7 118.73) (layer Dwgs.User)
+  (gr_text 1.25 (at 147.335 118.73) (layer F.CrtYd)
     (effects (font (size 1.5 1.5) (thickness 0.3)))
   )
-  (gr_circle (center 187.34 143.495) (end 188.44 143.495) (layer Edge.Cuts) (width 0.2))
-  (gr_circle (center 84.47 123.175) (end 85.57 123.175) (layer Edge.Cuts) (width 0.2))
-  (gr_circle (center 178.45 31.735) (end 179.55 31.735) (layer Edge.Cuts) (width 0.2))
-  (gr_circle (center 77.485 38.72) (end 78.585 38.72) (layer Edge.Cuts) (width 0.2))
-  (gr_arc (start 161.686 177.15) (end 204.612 140.066) (angle -65.01583871) (layer Dwgs.User) (width 0.2))
+  (gr_arc (start 161.305 171.435) (end 203.215 141.59) (angle -70.29569906) (layer Dwgs.User) (width 0.2))
   (gr_text "Designed by\n   @swan_match" (at 129.682 126.35) (layer B.SilkS)
     (effects (font (size 1.5 1.5) (thickness 0.3)) (justify mirror))
@@
   (gr_line (start 187.34 34.275) (end 187.34 113.015) (layer Edge.Cuts) (width 0.05))
   (gr_line (start 111.14 29.195) (end 182.26 29.195) (layer Edge.Cuts) (width 0.05))
-  (zone (net 0) (net_name "") (layer F.Cu) (hatch edge 0.508)
+  (zone (net 1) (net_name GND) (layer F.Cu) (hatch edge 0.508)
     (connect_pads (clearance 0.508))
     (min_thickness 0.254)
@@
     )
   )
-  (zone (net 0) (net_name "") (layer B.Cu) (hatch edge 0.508)
+  (zone (net 1) (net_name GND) (layer B.Cu) (hatch edge 0.508)
     (connect_pads (clearance 0.508))
     (min_thickness 0.254)
